Commit message: Sensor Lidar (ainda não funciona direito)

File: src/scout_description/urdf/scout_mini.xacro (robot description, xacro)
@@ -1,4 +1,10 @@
 <?xml version="1.0"?>
 <robot name="scout_mini" xmlns:xacro="http://ros.org/wiki/xacro">
+    <xacro:include filename="$(find scout_description)/urdf/lidar.xacro"/>
+    <material name="purple">
+        <color rgba="0.737 0.0 1.0 1" />
+    </material>
+    <!-- Lidar Sensor -->
+    <xacro:lidar/>
     <!-- Vehicle Geometries -->
     <!-- Base link -->
