Commit message: Lidar funcionando

File: src/scout_description/urdf/lidar.xacro (robot description, xacro)
@@ -4,10 +4,11 @@
    <xacro:macro name="lidar">
 	<joint name="laser_joint" type="fixed">
-	<parent link="base_link"/>
-	<child link="laser_frame"/>
-	<origin xyz="0.1 0 0.08" rpy="0 0 0"/>
+            <parent link="base_link"/>
+	    <child link="laser_frame"/>
+	    <origin xyz="0.1 0 0.08" rpy="0 0 0"/>
 	</joint>
 	<link name="laser_frame">
 	<visual>
+            <origin>"0.1 0 0.08"</origin>
 	    <geometry>
 	        <cylinder radius="0.05" length="0.04"/>
@@ -16,4 +17,5 @@
 	</visual>
 	<collision>
+            <origin>"0.1 0 0.08"</origin>
 	    <geometry>
 	        <cylinder radius="0.05" length="0.04"/>
@@ -31,10 +33,10 @@
 	    </material>
 	    <sensor name="laser" type="gpu_ray">
-	        <topic>"/scout_mini/scan"</topic>
-	        <pose> 0 0 0 0 0 0 </pose>
+	        <topic>/scout_mini/scan</topic>
+	        <pose> 0 0 0.2 0 0 0 </pose>
 	        <visualize>true</visualize>
 	        <update_rate>10</update_rate>
 	        <always_on>true</always_on>
-	        <gz_frame_id>"laser_frame"</gz_frame_id>
+	        <gz_frame_id>laser_frame</gz_frame_id>
 	        <ray>
 	            <scan>
